Commit message: Caster Wheel - Link & Joint

File: src/custom_bot/urdf/custom_bot.urdf (robot description, URDF)
Before this commit: robot custom_bot, 1 links, 0 joints
Links:
- added link caster_wheel; visual sphere radius=0.05
Joints:
- added joint caster_joint: type continuous, parent base_link, child caster_wheel, origin xyz=0.2 0 -0.05 rpy=0 0 0, axis 0 0 1
